File: OpenPrint.kicad_sch (KiCad schematic)
At the start: 52 parts, among them IC1 SN74AHCT1G125, IC2 100026223, J1 USB4215-03-A_REVA, U1 RP2354A, U2 AP2112K-3.3, U3 ATECC608C-MAHDA, U4 USBLC6-2SC6, Y1 ABM8-272-T3

Commit message: start routing
Parts:
- removed C18, C20, C22: 0.1uF, Capacitor_SMD:C_0402_1005Metric, symbol Device:C_Small
- removed D2, D3, D4: WS2812B, LED_SMD:LED_WS2812B_PLCC4_5.0x5.0mm_P3.2mm, symbol LED:WS2812B
- removed J1: USB4215-03-A_REVA, SamacSys_Parts:GCT_USB4215-03-A_REVA, symbol USB4215-03-A_REVA:USB4215-03-A_REVA
- added J2: USB4110-GF-A, USB4110-GF-A_GCT, symbol GCT4110:USB4110-GF-A
Connections:
- net GND: now also R12.2, J2.A1-B12 (GND), J2.A12-B1 (GND); no longer R12.1
- net RGB_DATA: now also U1.9 (GPIO6)
- net USB-CONN_DM: now also J2.A7 (DN1), J2.B7 (DN2)
- net USB-CONN_DP: now also J2.A6 (DP1), J2.B6 (DP2)
- net VBUS: now also J2.A4-B9 (VBUS), J2.A9-B4 (VBUS)
- net at R13.1: now also J2.B5 (CC2)
- new net: J2.A5 (CC1), R12.1
- no-connect marks 62 -> 61
Other:
- moved on the sheet: C14, C16, D1, IC1

Commit message: initial layout done
Parts:
- removed D1: WS2812B, LED_SMD:LED_WS2812B_PLCC4_5.0x5.0mm_P3.2mm, symbol LED:WS2812B
- removed J2: USB4110-GF-A, USB4110-GF-A_GCT, symbol GCT4110:USB4110-GF-A
- removed JP1, JP2: Jumper_2_Open, TestPoint:TestPoint_2Pads_Pitch2.54mm_Drill0.8mm, symbol Jumper:Jumper_2_Open
- removed R12: 5.1k, Resistor_SMD:R_0402_1005Metric, symbol Device:R
- added C19: 0.1uF, Capacitor_SMD:C_0402_1005Metric, symbol Device:C_Small
- added D1, D2: WS2812B-2020, LED_SMD:LED_WS2812B-2020_PLCC4_2.0x2.0mm, symbol LED:WS2812B-2020
- added H1, H2: MountingHole_Pad, MountingHole:MountingHole_2.2mm_M2_Pad, symbol Mechanical:MountingHole_Pad
- added H3, H4: MountingHole, MountingHole:MountingHole_2mm, symbol Mechanical:MountingHole
- added J1: USB4110, Connector_USB:USB_C_Receptacle_GCT_USB4110, symbol Connector:USB_C_Receptacle_USB2.0_16P
- added R14: 5.1k, Resistor_SMD:R_0402_1005Metric, symbol Device:R
- added S1, S2: SKRPABE010, SamacSys_Parts:SW_SKRPABE010, symbol SKRPABE010:SKRPABE010
- renumbered C23 to C1, C9 to C10, C10 to C12, C12 to C14, C17 to C16, C14 to C17, C16 to C18, C3 to C2, C19 to C20, C1 to C3, C2 to C4, C4 to C5, C5 to C6, C6 to C7, C7 to C9, R14 to R10, R10 to R11, R11 to R12, R9 to R6, R6 to R7, R7 to R8, R8 to R9, U3 to U1, U1 to U2, U4 to U3, U2 to U4
Connections:
- net BOOT: now also S2.3, S2.4
- net Earth: now also H1.1, H2.1, J1.SH (SHIELD)
- net GND: now also C19.1, D1.2 (VSS), D2.2 (VSS), J1.A1 (GND), J1.A12 (GND), J1.B1 (GND), J1.B12 (GND), R14.1, S1.1, S1.2, S2.1, S2.2
- net RST: no longer R1.1
- net USB-CONN_DM: now also U3.1 (I/O1), J1.A7 (D-), J1.B7 (D-); no longer U3.3 (I/O2)
- net USB-CONN_DP: now also U3.3 (I/O2), J1.A6 (D+), J1.B6 (D+); no longer U3.1 (I/O1)
- net USB-MCU_DM: now also U3.6 (I/O1); no longer U3.4 (I/O2)
- net USB-MCU_DP: now also U3.4 (I/O2); no longer U3.6 (I/O1)
- net VBUS: now also C19.2, D1.4 (VDD), D2.4 (VDD), J1.A4 (VBUS), J1.A9 (VBUS), J1.B4 (VBUS), J1.B9 (VBUS)
- net at R13.1: now also J1.A5 (CC1)
- net at IC1.4 (Y): now also D1.3 (DIN)
- new net: J1.B5 (CC2), R14.2
- new net: D1.1 (DOUT), D2.3 (DIN)
- new net RESET: R1.1, S1.3, S1.4
Other:
- note added: "Mounting Holes"
- moved on the sheet: C1, C17, C18, C20, C21, IC1, R6, U1, U4

Commit message: Route USB D- and update PCB layout
Renames USB D- nets consistently in the schematic and PCB, updates component placement and routing, and adds refined copper zones and fill settings for improved connectivity and clearance.
Connections:
- net USB-CONN_DM renamed USB-CONN_DN
- net USB-MCU_DM renamed USB-MCU_DN
Changed lines of the file:
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@@
 		)
 	)
-	(label "USB-CONN_DM"
+	(label "USB-CONN_DN"
 		(at 351.79 123.19 0)
 		(effects
@@
 		)
 	)
-	(label "USB-MCU_DM"
+	(label "USB-MCU_DN"
 		(at 63.5 123.19 180)
 		(effects
@@
 		)
 	)
-	(label "USB-CONN_DM"
+	(label "USB-CONN_DN"
 		(at 339.09 173.99 180)
 		(effects
@@
 		)
 	)
-	(label "USB-MCU_DM"
+	(label "USB-MCU_DN"
 		(at 354.33 173.99 0)
 		(effects
